File: 8X305/HW/8X305.kicad_sch (KiCad schematic)
At the start: 54 parts, among them J1 Conn_01x20, Q1 BC637, SW1 SW_Push, SW2 SW_Push, U1 8X305, U10 HY6116A, U11 NE555D, U12 DS8212D, U13 74LS175, U14 74LS40, U15 74HC244, U2 74HC74, U3 SST39SF010, U4 74LS175, U5 74LS175, U6 74LS04, U7 74LS175, U8 74LS175, U9 74LS03

Commit message: 8X305 madness!
Parts:
- added D7, D8, D9: LED, symbol Device:LED
- added R26, R27, R28: 1K, symbol Device:R
Connections:
- net GND: now also R26.2, R27.2, R28.2
- net at J1.20 (Pin_20), U13.11 (~{Q2}): now also D7.2 (A)
- net at J1.11 (Pin_11), U13.3 (~{Q0}): now also D9.2 (A)
- net at J1.16 (Pin_16), J1.18 (Pin_18), U13.6 (~{Q1}): now also D8.2 (A)
- new net: D9.1 (K), R28.1
- new net: D8.1 (K), R27.1
- new net: D7.1 (K), R26.1
